File: hardware/untitled.brd (EAGLE design)
At the start: 50.8 x 47.9 mm, 26 parts, among them IC1 ATSAMD21G18A-AU, IC2 IC_USBLC6-2, IC3 LM1117IMPX-3.3, J2 USB4110-GF-A, Y1 CRYSTAL-GROUNDEDSMD-5X3.2

Commit message: PCB updated
Parts:
- removed C27: (no value), rcl:C0603
- removed C62: (no value), rcl:SMC_A
- added C31: 100n, rcl:C0603
- added C6: (no value), rcl:C0402
- added D1: (no value), adafruit:SOD-323
- added JP3: (no value), pinhead:1X02
- added JP4: (no value), pinhead:1X03
- added L3: (no value), dp_devices:FB805
- added R13: 10k?, rcl:R0603
- added R7, R8: (no value), rcl:R0402
- added R9: (no value), rcl:R0603
- added T1, T2, T3: BC847, transistor:SOT23
- added U$2: SST25VF016BSO8M, mw:SO-08M
- R3, R4, R5: device rcl:R0603 -> rcl:R0402
- moved R4 8.42 mm to (26.2, 23.5), turned to 180 degrees
- moved JP2 8.29 mm to (14.1, 40.4)
- moved C1 8.28 mm to (18.5, 17.2)
- moved C14 8.28 mm to (36.7, 17.2)
- moved C3 8.28 mm to (22.7, 29.0)
- moved IC1 8.28 mm to (18.4, 24.8)
- moved IC2 8.28 mm to (31.4, 26.3)
- moved IC3 8.28 mm to (36.7, 11.0)
- moved J2 8.28 mm to (38.0, 26.3)
- moved R2 8.28 mm to (33.4, 28.9)
- moved Y1 8.28 mm to (20.9, 14.7)
- moved C10 8.28 mm to (20.0, 11.3)
- moved C15 8.28 mm to (31.4, 9.27)
- moved C2 8.28 mm to (21.8, 11.3)
- moved C4 8.28 mm to (19.0, 31.9)
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Connections:
- new net FLASH_CS: IC1.13, R13.1, U$2.1
- new net MISO: IC1.20, U$2.2
- new net MOSI: IC1.7, U$2.5
- new net N$10: R8.1, T2.3
- new net N$12: C6.1, IC1.6, L3.2
- new net N$3: R5.1, T1.1
- new net N$4: D1.A, JP3.2, T1.3
- new net N$5: R4.1, T2.1
- new net N$6: R3.1, T3.1
- new net N$7: JP4.3, R7.2
- new net N$8: R7.1, T3.3
- new net N$9: JP4.2, R8.2
- new net SC3V3: D1.C, JP3.1, R9.1
- new net SCK: IC1.8, U$2.6
- net 3V3: now also C31.1, JP4.1, L3.1, R13.2, R9.2, U$2.3, U$2.7, U$2.8
- net 5V: no longer C62.+
- net GND: now also C31.2, C6.2, T1.2, T2.2, T3.2, U$2.4; no longer C27.2, C62.-
- net VBUS: no longer C27.1
Routing:
- net 3V3: track 43.2 -> 113.0 mm, vias 0 -> 2
- net N$5: track 0.00 -> 17.8 mm, vias 0 -> 1
- net N$6: track 0.00 -> 16.1 mm, vias 0 -> 1
- net MISO: track 0.00 -> 16.0 mm
- net FLASH_CS: track 0.00 -> 13.1 mm
- net SCK: track 0.00 -> 9.08 mm
- net N$12: track 0.00 -> 9.05 mm
- net N$10: track 0.00 -> 7.92 mm, vias 0 -> 1
- net MOSI: track 0.00 -> 7.84 mm
- net N$4: track 0.00 -> 5.32 mm
- net SC3V3: track 0.00 -> 5.29 mm
- net N$3: track 0.00 -> 4.98 mm
- net GND: track 12.5 -> 17.1 mm, vias 7 -> 12
- net N$7: track 0.00 -> 3.84 mm
- net N$9: track 0.00 -> 2.60 mm
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Other:
- board size 50.8 x 47.9 mm -> 42.5 x 47.9 mm

Commit message: Mounting holes added to PCB
Other:
- board size 42.5 x 47.9 mm -> 42.5 x 47.6 mm
Changed lines of the file:
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@@
 <setting verticaltext="up"/>
 </settings>
-<grid distance="25" unitdist="mil" unit="mil" style="lines" multiple="1" display="no" altdistance="1" altunitdist="mil" altunit="mil"/>
+<grid distance="25" unitdist="mil" unit="mil" style="lines" multiple="1" display="no" altdistance="5" altunitdist="mil" altunit="mil"/>
 <layers>
 <layer number="1" name="Top" color="4" fill="1" visible="yes" active="yes"/>
@@
 <plain>
 <wire x1="0" y1="0" x2="42.525" y2="0" width="0" layer="20"/>
-<wire x1="42.525" y1="0" x2="42.525" y2="47.93" width="0" layer="20"/>
-<wire x1="42.525" y1="47.93" x2="0" y2="47.93" width="0" layer="20"/>
-<wire x1="0" y1="47.93" x2="0" y2="0" width="0" layer="20"/>
+<wire x1="42.525" y1="0" x2="42.525" y2="47.625" width="0" layer="20"/>
+<wire x1="42.525" y1="47.625" x2="0" y2="47.625" width="0" layer="20"/>
+<wire x1="0" y1="47.625" x2="0" y2="0" width="0" layer="20"/>
 <rectangle x1="33.441640625" y1="16.7132" x2="35.245034375" y2="18.59025625" layer="41"/>
+<hole x="39.29" y="3.095" drill="2"/>
+<circle x="39.29" y="3.095" radius="3.048" width="0" layer="41"/>
+<circle x="39.29" y="3.095" radius="3.048" width="0" layer="42"/>
+<hole x="3.095" y="3.095" drill="2"/>
+<circle x="3.095" y="3.095" radius="3.048" width="0" layer="41"/>
+<circle x="3.095" y="3.095" radius="3.048" width="0" layer="42"/>
+<hole x="3.095" y="44.37" drill="2"/>
+<circle x="3.095" y="44.37" radius="3.048" width="0" layer="41"/>
+<circle x="3.095" y="44.37" radius="3.048" width="0" layer="42"/>
+<hole x="39.29" y="44.37" drill="2"/>
+<circle x="39.29" y="44.37" radius="3.048" width="0" layer="41"/>
+<circle x="39.29" y="44.37" radius="3.048" width="0" layer="42"/>
 </plain>
 <attributes>
@@
 <wire x1="10.9474" y1="25.5524" x2="10.9474" y2="31.154" width="0.4064" layer="1"/>
 </signal>
+<signal name="N$13">
+<via x="39.29" y="3.095" extent="1-16" drill="0.6" diameter="1.27"/>
+</signal>
+<signal name="N$11">
+<via x="3.095" y="3.095" extent="1-16" drill="0.6" diameter="1.27"/>
+</signal>
+<signal name="N$14">
+<via x="3.095" y="44.37" extent="1-16" drill="0.6" diameter="1.27"/>
+</signal>
+<signal name="N$15">
+<via x="39.29" y="44.37" extent="1-16" drill="0.6" diameter="1.27"/>
+</signal>
 </signals>

Commit message: PCB updated
Parts:
- added D2, D3: (no value), adafruit:SOD-323
- added F2: 1206L012, polyfuse-smd_10:1206L
- added JP5: (no value), pinhead:1X04
- added Q3: BSS123, transistor-small-signal:SOT23
- added R10: (no value), rcl:R0402
- added R11, R12: (no value), rcl:R0603
- moved JP2 4.04 mm to (11.5, 37.3)
Connections:
- new net LOCK: IC1.37, R10.2
- new net LOCK_5V: D3.C, F2.1, JP5.3
- new net LOCK_OPEN: D2.C, IC1.38, JP5.1, R12.1
- new net N$16: Q3.1, R10.1, R11.1
- new net N$17: D3.A, JP5.2, Q3.3
- net 3V3: now also R12.2
- net GND: now also D2.A, JP5.4, Q3.2, R11.2
- net VBUS: now also F2.2
Routing:
- net LOCK_OPEN: track 0.00 -> 14.4 mm
- net LOCK_5V: track 0.00 -> 6.42 mm
- net N$17: track 0.00 -> 5.32 mm
- net VBUS: track 26.6 -> 30.8 mm
- net LOCK: track 0.00 -> 3.52 mm
- net 3V3: track 113.0 -> 109.7 mm
- net N$16: track 0.00 -> 3.14 mm
- net SWCLK: track 21.2 -> 18.4 mm
- net SWDIO: track 11.4 -> 9.39 mm
- net GND: track 17.1 -> 17.6 mm, vias 12 -> 15
Other:
- board size 42.5 x 47.6 mm -> 42.5 x 44.5 mm
