File: hardware/untitled.sch (EAGLE design)
At the start: 26 parts, among them IC1 ATSAMD21G18A-AU, IC2 IC_USBLC6-2, IC3 LM1117IMPX-3.3, J2 USB4110-GF-A, Y1 CRYSTAL-GROUNDEDSMD-5X3.2

Commit message: PCB updated
Parts:
- removed C27: (no value), rcl:C-EUC0603
- removed C62: (no value), rcl:CPOL-EUSMCA
- added C31: 100n, rcl:C-EUC0603
- added C6: (no value), rcl:C-EUC0402
- added D1: (no value), adafruit:DIODESOD-323
- added JP3: (no value), pinhead:PINHD-1X2
- added JP4: (no value), pinhead:PINHD-1X3
- added L3: (no value), dp_devices:FERRITE-0805
- added R13: 10k?, rcl:R-EU_R0603
- added R7, R8: (no value), rcl:R-EU_R0402
- added R9: (no value), rcl:R-EU_R0603
- added T1, T2, T3: BC847, transistor:BC847
- added U$2: SST25VF016BSO8M, mw:SST25VF016BSO8M
- R3, R4, R5: device rcl:R-EU_R0603 -> rcl:R-EU_R0402
Connections:
- new net FLASH_CS: IC1.PA08, R13.1, U$2.!CE
- new net MISO: IC1.PB11, U$2.SO
- new net MOSI: IC1.PB08, U$2.SI
- new net N$10: R8.1, T2.C
- new net N$12: C6.1, IC1.VDDANA, L3.2
- new net N$3: R5.1, T1.B
- new net N$4: D1.A, JP3.2, T1.C
- new net N$5: R4.1, T2.B
- new net N$6: R3.1, T3.B
- new net N$7: JP4.3, R7.2
- new net N$8: R7.1, T3.C
- new net N$9: JP4.2, R8.2
- new net SC3V3: D1.C, JP3.1, R9.1
- new net SCK: IC1.PB09, U$2.SCK
- net 3V3: now also C31.1, JP4.1, L3.1, R13.2, R9.2, U$2.!HOLD, U$2.!WP, U$2.VDD
- net 5V: no longer C62.+
- net GND: now also C31.2, C6.2, T1.E, T2.E, T3.E, U$2.VSS; no longer C27.2, C62.-
- net VBUS: no longer C27.1
Other:
- moved on the sheet: R3, R4

Commit message: PCB updated
Parts:
- added D2, D3: (no value), adafruit:DIODESOD-323
- added F2: 1206L012, polyfuse-smd_10:1206L012
- added JP5: (no value), pinhead:PINHD-1X4
- added Q3: BSS123, transistor-small-signal:BSS123
- added R10: (no value), rcl:R-EU_R0402
- added R11, R12: (no value), rcl:R-EU_R0603
Connections:
- new net LOCK: IC1.PB22, R10.2
- new net LOCK_5V: D3.C, F2.1, JP5.3
- new net LOCK_OPEN: D2.C, IC1.PB23, JP5.1, R12.1
- new net N$16: Q3.G, R10.1, R11.1
- new net N$17: D3.A, JP5.2, Q3.D
- net 3V3: now also R12.2
- net GND: now also D2.A, JP5.4, Q3.S, R11.2
- net VBUS: now also F2.2
Changed lines of the file:
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@@
 <part name="C6" library="rcl" deviceset="C-EU" device="C0402"/>
 <part name="GND4" library="supply1" deviceset="GND" device=""/>
+<part name="F2" library="polyfuse-smd_10" deviceset="?" device="1206L" technology="012" value="1206L012"/>
+<part name="Q3" library="transistor-small-signal" deviceset="BSS123" device=""/>
+<part name="GND21" library="supply1" deviceset="GND" device=""/>
+<part name="R10" library="rcl" deviceset="R-EU_" device="R0402"/>
+<part name="JP5" library="pinhead" deviceset="PINHD-1X4" device=""/>
+<part name="GND22" library="supply1" deviceset="GND" device=""/>
+<part name="R11" library="rcl" deviceset="R-EU_" device="R0603"/>
+<part name="GND24" library="supply1" deviceset="GND" device=""/>
+<part name="D3" library="adafruit" deviceset="DIODE" device="SOD-323"/>
+<part name="R12" library="rcl" deviceset="R-EU_" device="R0603"/>
+<part name="D2" library="adafruit" deviceset="DIODE" device="SOD-323"/>
+<part name="GND25" library="supply1" deviceset="GND" device=""/>
 </parts>
 <sheets>
@@
 <instance part="C6" gate="G$1" x="22.86" y="35.56"/>
 <instance part="GND4" gate="1" x="22.86" y="25.4"/>
+<instance part="F2" gate="G$1" x="-55.88" y="251.46" rot="R90"/>
+<instance part="Q3" gate="G$1" x="154.94" y="187.96"/>
+<instance part="GND21" gate="1" x="154.94" y="167.64"/>
+<instance part="R10" gate="G$1" x="139.7" y="185.42" rot="R180"/>
+<instance part="JP5" gate="A" x="170.18" y="200.66"/>
+<instance part="GND22" gate="1" x="160.02" y="167.64"/>
+<instance part="R11" gate="G$1" x="147.32" y="177.8" rot="R270"/>
+<instance part="GND24" gate="1" x="147.32" y="167.64"/>
+<instance part="D3" gate="G$1" x="149.86" y="200.66" rot="R90"/>
+<instance part="R12" gate="G$1" x="144.78" y="213.36" rot="R90"/>
+<instance part="D2" gate="G$1" x="144.78" y="200.66" rot="R90"/>
+<instance part="GND25" gate="1" x="144.78" y="193.04"/>
 </instances>
 <busses>
@@
 <pinref part="GND4" gate="1" pin="GND"/>
 <wire x1="22.86" y1="27.94" x2="22.86" y2="30.48" width="0.1524" layer="91"/>
+</segment>
+<segment>
+<pinref part="Q3" gate="G$1" pin="S"/>
+<pinref part="GND21" gate="1" pin="GND"/>
+<wire x1="154.94" y1="170.18" x2="154.94" y2="182.88" width="0.1524" layer="91"/>
+</segment>
+<segment>
+<pinref part="JP5" gate="A" pin="4"/>
+<pinref part="GND22" gate="1" pin="GND"/>
+<wire x1="167.64" y1="198.12" x2="160.02" y2="198.12" width="0.1524" layer="91"/>
+<wire x1="160.02" y1="198.12" x2="160.02" y2="170.18" width="0.1524" layer="91"/>
+</segment>
+<segment>
+<pinref part="R11" gate="G$1" pin="2"/>
+<pinref part="GND24" gate="1" pin="GND"/>
+<wire x1="147.32" y1="170.18" x2="147.32" y2="172.72" width="0.1524" layer="91"/>
+</segment>
+<segment>
+<pinref part="D2" gate="G$1" pin="A"/>
+<pinref part="GND25" gate="1" pin="GND"/>
+<wire x1="144.78" y1="195.58" x2="144.78" y2="198.12" width="0.1524" layer="91"/>
 </segment>
 </net>
@@
 <pinref part="F1" gate="G$1" pin="1"/>
 <wire x1="-50.8" y1="241.3" x2="-55.88" y2="241.3" width="0.1524" layer="91"/>
+<pinref part="F2" gate="G$1" pin="2"/>
+<wire x1="-55.88" y1="241.3" x2="-63.5" y2="241.3" width="0.1524" layer="91"/>
+<wire x1="-55.88" y1="246.38" x2="-55.88" y2="241.3" width="0.1524" layer="91"/>
+<junction x="-55.88" y="241.3"/>
 </segment>
 </net>
@@
 <pinref part="IC1" gate="G$1" pin="PA18"/>
 <wire x1="81.28" y1="35.56" x2="88.9" y2="35.56" width="0.1524" layer="91"/>
+<label x="88.9" y="35.56" size="1.4224" layer="95" xref="yes"/>
 </segment>
 <segment>
@@
 <pinref part="IC1" gate="G$1" pin="PA19"/>
 <wire x1="81.28" y1="38.1" x2="88.9" y2="38.1" width="0.1524" layer="91"/>
+<label x="88.9" y="38.1" size="1.4224" layer="95" xref="yes"/>
 </segment>
 <segment>
@@
 <wire x1="83.82" y1="66.04" x2="83.82" y2="58.42" width="0.1524" layer="91"/>
 <junction x="83.82" y="58.42"/>
+<label x="91.44" y="58.42" size="1.4224" layer="95" xref="yes"/>
 </segment>
 <segment>
@@
 <wire x1="22.86" y1="66.04" x2="22.86" y2="71.12" width="0.1524" layer="91"/>
 </segment>
+<segment>
+<pinref part="R12" gate="G$1" pin="2"/>
+<wire x1="144.78" y1="218.44" x2="144.78" y2="220.98" width="0.1524" layer="91"/>
+</segment>
 </net>
 <net name="TX" class="0">
@@
 <pinref part="IC1" gate="G$1" pin="PA10"/>
 <wire x1="50.8" y1="10.16" x2="50.8" y2="5.08" width="0.1524" layer="91"/>
+<label x="50.8" y="5.08" size="1.4224" layer="95" rot="R270" xref="yes"/>
 </segment>
 <segment>
@@
 <pinref part="IC1" gate="G$1" pin="PA11"/>
 <wire x1="53.34" y1="10.16" x2="53.34" y2="5.08" width="0.1524" layer="91"/>
+<label x="53.34" y="5.08" size="1.4224" layer="95" rot="R270" xref="yes"/>
 </segment>
 <segment>
@@
 <pinref part="IC1" gate="G$1" pin="PB09"/>
 <wire x1="38.1" y1="40.64" x2="30.48" y2="40.64" width="0.1524" layer="91"/>
+<label x="30.48" y="40.64" size="1.4224" layer="95" rot="R180" xref="yes"/>
 </segment>
 </net>
@@
 <pinref part="IC1" gate="G$1" pin="PB11"/>
 <wire x1="63.5" y1="10.16" x2="63.5" y2="5.08" width="0.1524" layer="91"/>
+<label x="63.5" y="5.08" size="1.4224" layer="95" rot="R270" xref="yes"/>
 </segment>
 </net>
@@
 <pinref part="IC1" gate="G$1" pin="PB08"/>
 <wire x1="38.1" y1="43.18" x2="30.48" y2="43.18" width="0.1524" layer="91"/>
+<label x="30.48" y="43.18" size="1.4224" layer="95" rot="R180" xref="yes"/>
 </segment>
 </net>
@@
 <pinref part="IC1" gate="G$1" pin="PA08"/>
 <wire x1="45.72" y1="10.16" x2="45.72" y2="5.08" width="0.1524" layer="91"/>
+<label x="45.72" y="5.08" size="1.4224" layer="95" rot="R270" xref="yes"/>
 </segment>
 </net>
@@
 </segment>
 </net>
+<net name="N$16" class="0">
+<segment>
+<pinref part="Q3" gate="G$1" pin="G"/>
+<pinref part="R10" gate="G$1" pin="1"/>
+<wire x1="149.86" y1="185.42" x2="147.32" y2="185.42" width="0.1524" layer="91"/>
+<pinref part="R11" gate="G$1" pin="1"/>
+<wire x1="147.32" y1="185.42" x2="144.78" y2="185.42" width="0.1524" layer="91"/>
+<wire x1="147.32" y1="182.88" x2="147.32" y2="185.42" width="0.1524" layer="91"/>
+<junction x="147.32" y="185.42"/>
+</segment>
+</net>
+<net name="N$17" class="0">
+<segment>
+<pinref part="Q3" gate="G$1" pin="D"/>
+<wire x1="154.94" y1="203.2" x2="154.94" y2="195.58" width="0.1524" layer="91"/>
+<pinref part="JP5" gate="A" pin="2"/>
+<wire x1="154.94" y1="195.58" x2="154.94" y2="193.04" width="0.1524" layer="91"/>
+<wire x1="167.64" y1="203.2" x2="154.94" y2="203.2" width="0.1524" layer="91"/>
+<wire x1="149.86" y1="198.12" x2="149.86" y2="195.58" width="0.1524" layer="91"/>
+<wire x1="149.86" y1="195.58" x2="154.94" y2="195.58" width="0.1524" layer="91"/>
+<junction x="154.94" y="195.58"/>
+<pinref part="D3" gate="G$1" pin="A"/>
+</segment>
+</net>
+<net name="LOCK_5V" class="0">
+<segment>
+<pinref part="F2" gate="G$1" pin="1"/>
+<wire x1="-55.88" y1="256.54" x2="-55.88" y2="259.08" width="0.1524" layer="91"/>
+</segment>
+<segment>
+<pinref part="JP5" gate="A" pin="3"/>
+<wire x1="167.64" y1="200.66" x2="160.02" y2="200.66" width="0.1524" layer="91"/>
+<wire x1="160.02" y1="200.66" x2="160.02" y2="208.28" width="0.1524" layer="91"/>
+<wire x1="160.02" y1="208.28" x2="160.02" y2="213.36" width="0.1524" layer="91"/>
+<wire x1="160.02" y1="208.28" x2="149.86" y2="208.28" width="0.1524" layer="91"/>
+<wire x1="149.86" y1="208.28" x2="149.86" y2="203.2" width="0.1524" layer="91"/>
+<junction x="160.02" y="208.28"/>
+<pinref part="D3" gate="G$1" pin="C"/>
+</segment>
+</net>
+<net name="LOCK" class="0">
+<segment>
+<pinref part="R10" gate="G$1" pin="2"/>
+<wire x1="134.62" y1="185.42" x2="132.08" y2="185.42" width="0.1524" layer="91"/>
+</segment>
+<segment>
+<pinref part="IC1" gate="G$1" pin="PB22"/>
+<wire x1="73.66" y1="78.74" x2="73.66" y2="91.44" width="0.1524" layer="91"/>
+</segment>
+</net>
+<net name="LOCK_OPEN" class="0">
+<segment>
+<pinref part="IC1" gate="G$1" pin="PB23"/>
+<wire x1="71.12" y1="78.74" x2="71.12" y2="91.44" width="0.1524" layer="91"/>
+</segment>
+<segment>
+<pinref part="JP5" gate="A" pin="1"/>
+<wire x1="167.64" y1="205.74" x2="144.78" y2="205.74" width="0.1524" layer="91"/>
+<pinref part="R12" gate="G$1" pin="1"/>
+<wire x1="144.78" y1="205.74" x2="137.16" y2="205.74" width="0.1524" layer="91"/>
+<wire x1="144.78" y1="208.28" x2="144.78" y2="205.74" width="0.1524" layer="91"/>
+<junction x="144.78" y="205.74"/>
+<pinref part="D2" gate="G$1" pin="C"/>
+<wire x1="144.78" y1="203.2" x2="144.78" y2="205.74" width="0.1524" layer="91"/>
+</segment>
+</net>
